Commit message: Added launch file and updated some stuffz.

File: models/navvis.urdf (robot description, URDF)
Before this commit: robot Navvis, 9 links, 8 joints
Links:
- link base: geometry collision box size=0.94 0.78 1.98; visual box size=0.2 0.3 1.80
Joints:
- joint base2wheel_front_left: axis (none) -> 0 1 0; limit (none) -> effort=.1 velocity=99; type fixed -> continuous
- joint base2wheel_front_right: axis (none) -> 0 1 0; limit (none) -> effort=.1 velocity=99; type fixed -> continuous
- joint base2wheel_left: axis (none) -> 0 1 0; limit (none) -> effort=.1 velocity=99; type fixed -> continuous
- joint base2wheel_right: axis (none) -> 0 1 0; limit (none) -> effort=.1 velocity=99; type fixed -> continuous

File: models/navvis.xacro (robot description, xacro)
@@ -41,5 +41,5 @@
 			</collision>
 		</link>
-		<joint name="base2wheel_${description}" type="revolute">
+		<joint name="base2wheel_${description}" type="continuous">
 			<parent link="base" />
 			<child link="wheel_${description}"/>

Commit message: Gave the lasers more accurate meshes and added README

File: models/navvis.urdf (robot description, URDF)
Before this commit: robot Navvis, 9 links, 8 joints
Links:
- removed link laser_vert_bottom
- removed link laser_vert_top_left
- removed link laser_vert_top_right
- added link bottom, mass 1e-5; collision box size=0.1 0.1 0.1; visual mesh filename=package://gazebo_plugins/test/multi_robot_scenario/meshes/l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
- added link laser_horiz_base_link, mass 0.83; collision cylinder length=0.0717 radius=0.0516; visual mesh filename=package://velodyne_description/meshes/VLP16_base_1.dae
- added link top_left, mass 1e-5; collision box size=0.1 0.1 0.1; visual mesh filename=package://gazebo_plugins/test/multi_robot_scenario/meshes/l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
- added link top_right, mass 1e-5; collision box size=0.1 0.1 0.1; visual mesh filename=package://gazebo_plugins/test/multi_robot_scenario/meshes/l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
- link laser_horiz: mass None -> 0.01; geometry visual mesh filename=package://velodyne_description/meshes/VLP16_scan.dae
Joints:
- removed joint base2laser_horiz
- removed joint base2laser_vert_bottom
- removed joint base2laser_vert_top_left
- removed joint base2laser_vert_top_right
- added joint base_bottom_joint: type fixed, parent base, child bottom, origin xyz=0.3158 -0.0021 .51 rpy=3.1355 -1.3045 0.0025, axis 0 0 1
- added joint base_top_left_joint: type fixed, parent base, child top_left, origin xyz=0.2997 0.1531 1.8443 rpy=1.178 0.6198 1.9560, axis 0 0 1
- added joint base_top_right_joint: type fixed, parent base, child top_right, origin xyz=0.2978 -0.1450 1.8451 rpy=-1.176 0.6313 -1.9377, axis 0 0 1
- added joint laser_horiz_base_mount_joint: type fixed, parent base, child laser_horiz_base_link, origin xyz=0.2325416305773505 -0.0001380069427607134 1.920122926231907 rpy=-0.0012068 0.114646 -0.0015308
- added joint laser_horiz_base_scan_joint: type fixed, parent laser_horiz_base_link, child laser_horiz, origin xyz=0 0 0.0377 rpy=0 0 0

File: models/navvis.xacro (robot description, xacro)
@@ -1,4 +1,6 @@
 <?xml version="1.0"?>
 <robot xmlns:xacro="https://www.ros.org/wiki/xacro" name="Navvis" >
+	<xacro:include filename="$(find gazebo_plugins)/test/multi_robot_scenario/xacro/laser/hokuyo.xacro" />
+	<xacro:include filename="$(find velodyne_description)/urdf/VLP-16.urdf.xacro" />
 	<material name="white">
 		<color rgba="1 1 1 1"/>
@@ -71,5 +73,5 @@
 			</collision>
 	</link>
-	<link name="laser_horiz">
+	<!--link name="laser_horiz">
 			<visual>
 				<material name="black"/>
@@ -87,5 +89,12 @@
 	<xacro:laser_vert description="top_right" xyz="0.2978 -0.1450 1.8451" rpy="-1.176 0.6313 -1.9377"/>
 	<xacro:laser_vert description="top_left" xyz="0.2997 0.1531 1.8443" rpy="1.178 0.6198 1.9560"/>
-	<xacro:laser_vert description="bottom" xyz="0.3158 -0.0021 .51" rpy="3.1355 -1.3045 0.0025"/>
+	<xacro:laser_vert description="bottom" xyz="0.3158 -0.0021 .51" rpy="3.1355 -1.3045 0.0025"/-->
+	<VLP-16 parent="base" name="laser_horiz" topic="laser_horiz/packets" hz="10" samples="440" gpu="false">
+		<origin xyz="0.2325416305773505 -0.0001380069427607134 1.920122926231907"
+rpy="-0.0012068 0.114646 -0.0015308" />
+	</VLP-16>
+	<xacro:laser name="top_right" parent="base" xyz="0.2978 -0.1450 1.8451" rpy="-1.176 0.6313 -1.9377" meshes="package://gazebo_plugins/test/multi_robot_scenario/meshes/laser" />
+	<xacro:laser name="top_left" parent="base" xyz="0.2997 0.1531 1.8443" rpy="1.178 0.6198 1.9560" meshes="package://gazebo_plugins/test/multi_robot_scenario/meshes/laser" />
+	<xacro:laser name="bottom" parent="base" xyz="0.3158 -0.0021 .51" rpy="3.1355 -1.3045 0.0025" meshes="package://gazebo_plugins/test/multi_robot_scenario/meshes/laser" />
 	<xacro:wheel description="right" xyz="-0.1 -0.4 .2" radius=".2"/>
 	<xacro:wheel description="left" xyz="-0.1 0.4 .2" radius=".2"/>
